Commit message: variable names updates

File: tas_car_description/urdf/macros.xacro (robot description, xacro)
@@ -39,10 +39,10 @@
             <inertial>
                 <origin xyz="0 0 0" rpy="${PI/2} 0 0" />
-                <mass value="${wheelMass}"/>
+                <mass value="${wheel_mass}"/>
                 <cylinder_inertia m="${axle_mass}" r="${axle_radius}" h="${axle_length}"/>
             </inertial>
         </link>
         <joint name="${fr_prefix}_axle_joint" type="fixed">
-            <origin xyz="${fr_position * chassisLength / 2} 0 ${wheelRadius + chassisHeight/2}" rpy="0 0 0" />
+            <origin xyz="${fr_position * chassis_length / 2} 0 ${wheel_radius + chassis_height/2}" rpy="0 0 0" />
             <parent link="chassis"/>
             <child link="${fr_prefix}_axle"/>
@@ -56,5 +56,5 @@
                 <origin xyz="0 0 0" rpy="0 0 ${PI/2}" />
                 <geometry>
-                    <cylinder length="${wheelWidth}" radius="${wheelRadius}"/>
+                    <cylinder length="${wheel_width}" radius="${wheel_radius}"/>
                 </geometry>
             </collision>
@@ -62,5 +62,5 @@
                 <origin xyz="0 0 0" rpy="0 ${PI/2} ${PI/2}" />
                 <geometry>
-                    <cylinder length="${wheelWidth}" radius="${wheelRadius}"/>
+                    <cylinder length="${wheel_width}" radius="${wheel_radius}"/>
                 </geometry>
                 <material name="black"/>
@@ -68,6 +68,6 @@
             <inertial>
                 <origin xyz="0 0 0" rpy="0 ${PI/2} ${PI/2}" />
-                <mass value="${wheelMass}"/>
-                <cylinder_inertia m="${wheelMass}" r="${wheelRadius}" h="${wheelWidth}"/>
+                <mass value="${wheel_mass}"/>
+                <cylinder_inertia m="${wheel_mass}" r="${wheel_radius}" h="${wheel_width}"/>
             </inertial>
             <max_contacts>1</max_contacts>
@@ -141,8 +141,9 @@
                 <parent link="${fr_prefix}_${lr_prefix}_wheel_carrier" />
                 <child link="${fr_prefix}_${lr_prefix}_wheel"/>
-                <origin xyz="0 ${lr_position*(wheelWidth/2)} 0" ryp="0 0 0" />
+                <origin xyz="0 ${lr_position*(wheel_width/2)} 0" ryp="0 0 0" />
                 <axis xyz="0 1 0" rpy="0 0 0" />
                 <limit effort="${axle_eff_limit}" velocity="${axle_vel_limit}"/>
-                <dynamics damping="0.001" friction="0.5"/>
+                <!-- Damping and friction of the joint. -->
+                <dynamics damping="0.5" friction="1.5"/>
             </joint>
             <transmission name="${fr_prefix}_${lr_prefix}_trans">
@@ -172,5 +173,5 @@
             <parent link="${fr_prefix}_axle"/>
             <child link="${fr_prefix}_${lr_prefix}_wheel"/>
-            <origin xyz="0 ${lr_position*(axle_length/2) + lr_position*(wheelWidth/2)} 0" ryp="0 0 0" />
+            <origin xyz="0 ${lr_position*(axle_length/2) + lr_position*(wheel_width/2)} 0" ryp="0 0 0" />
             <!-- Add -0.01 to align the wheels. -->
             <axis xyz="0 1 0" rpy="0 0 0" />

File: tas_car_description/urdf/tas_car.xacro (robot description, xacro)
@@ -5,16 +5,16 @@
         <xacro:property name="PI" value="3.1415926535897931"/>
         <!-- Chassis. -->
-		<xacro:property name="chassisLength" value="0.358"/>
-		<xacro:property name="chassisWidth" value="0.18"/>
-		<xacro:property name="chassisHeight" value="0.068"/> <!-- Almin: 0.138 -->
-		<xacro:property name="chassisMass" value="3"/>
+		<xacro:property name="chassis_length" value="0.358"/>
+		<xacro:property name="chassis_width" value="0.18"/>
+		<xacro:property name="chassis_height" value="0.068"/> <!-- Almin: 0.138 -->
+		<xacro:property name="chassis_mass" value="3"/>
 		<!-- Caster. -->
 		<xacro:property name="casterRadius" value="0.05"/>
 		<xacro:property name="casterMass" value="5"/>
 		<!-- Wheels. -->
-		<xacro:property name="wheelWidth" value="0.059"/>
-		<xacro:property name="wheelRadius" value="0.0695"/>
-		<xacro:property name="wheelPos" value="0.179"/>
-		<xacro:property name="wheelMass" value="0.5"/>
+		<xacro:property name="wheel_width" value="0.059"/>
+		<xacro:property name="wheel_radius" value="0.0695"/>
+		<xacro:property name="wheel_pos" value="0.179"/>
+		<xacro:property name="wheel_mass" value="0.5"/>
 		<xacro:property name="wheelOffsetX" value="0.179" />
 		<xacro:property name="wheelOffsetY" value="0.1815" />
@@ -35,20 +35,20 @@
 		<link name="chassis">
 			<collision>
-				<origin xyz="0 0 ${wheelRadius}" rpy="0 0 0"/>
+				<origin xyz="0 0 ${wheel_radius}" rpy="0 0 0"/>
 			    <geometry>
-			      <box size="${chassisLength} ${chassisWidth} ${chassisHeight}"/>
+			      <box size="${chassis_length} ${chassis_width} ${chassis_height}"/>
 			    </geometry>
 			</collision>
 			<visual>
-				<origin xyz="0 0 ${wheelRadius}" rpy="0 0 0"/>
+				<origin xyz="0 0 ${wheel_radius}" rpy="0 0 0"/>
 			    <geometry>
-			    	<box size="${chassisLength} ${chassisWidth} ${chassisHeight}"/>
+			    	<box size="${chassis_length} ${chassis_width} ${chassis_height}"/>
 			    </geometry>
 			    <material name="orange"/>
 			</visual>
 			<inertial>
-				<origin xyz="0 0 ${wheelRadius}" rpy="0 0 0"/>
-      			<mass value="${chassisMass}"/>
-      			<box_inertia m="${chassisMass}" x="${chassisLength}" y="${chassisWidth}" z="${chassisHeight}"/>
+				<origin xyz="0 0 ${wheel_radius}" rpy="0 0 0"/>
+      			<mass value="${chassis_mass}"/>
+      			<box_inertia m="${chassis_mass}" x="${chassis_length}" y="${chassis_width}" z="${chassis_height}"/>
 			</inertial>
 		</link>
@@ -62,5 +62,5 @@
 	<!--
 		<joint name="camera_joint" type="fixed">
-			<origin xyz="${-cameraSize+chassisLength/2} 0 ${cameraSize+wheelRadius+cameraSize/2}" rpy="0 0 0"/>
+			<origin xyz="${-cameraSize+chassis_length/2} 0 ${cameraSize+wheel_radius+cameraSize/2}" rpy="0 0 0"/>
 			<parent link="chassis"/>
 			<child link="camera"/>
@@ -90,5 +90,5 @@
 		<joint name="hokuyo_joint" type="fixed">
 			<axis xyz="0 1 0" />
-			<origin xyz="${-cameraSize+chassisLength/2} 0 ${cameraSize+wheelRadius}" rpy="0 0 0"/>
+			<origin xyz="${-cameraSize+chassis_length/2} 0 ${cameraSize+wheel_radius}" rpy="0 0 0"/>
 			<parent link="chassis"/>
 			<child link="hokuyo_link"/>

File: tas_car_description/urdf/tas_car_platform.urdf.xacro (robot description, xacro)
@@ -8,10 +8,10 @@
         <xacro:property name="PI" value="3.1415926535897931"/>
         <!-- Chassis. -->
-        <xacro:property name="chassisLength" value="0.358"/>
-        <xacro:property name="chassisWidth" value="0.18"/>
-        <xacro:property name="chassisHeight" value="0.068"/>
-        <xacro:property name="chassisMass" value="3"/>
+        <xacro:property name="chassis_length" value="0.358"/>
+        <xacro:property name="chassis_width" value="0.18"/>
+        <xacro:property name="chassis_height" value="0.068"/>
+        <xacro:property name="chassis_mass" value="3"/>
         <!-- Axle. -->
-        <xacro:property name="axle_length" value="${chassisWidth + 0.02}" />
+        <xacro:property name="axle_length" value="${chassis_width + 0.02}" />
         <xacro:property name="axle_radius" value="0.01" />
         <xacro:property name="axle_mass" value="0.2" />
@@ -28,8 +28,8 @@
         <xacro:property name="servo_no_load_speed" value="8.05536578" />
         <!-- Wheels. -->
-        <xacro:property name="wheelWidth" value="0.059"/>
-        <xacro:property name="wheelRadius" value="0.0695"/>
-        <xacro:property name="wheelPos" value="0.179"/>
-        <xacro:property name="wheelMass" value="0.5"/>
+        <xacro:property name="wheel_width" value="0.059"/>
+        <xacro:property name="wheel_radius" value="0.0695"/>
+        <xacro:property name="wheel_pos" value="0.179"/>
+        <xacro:property name="wheel_mass" value="0.5"/>
         <xacro:property name="wheelOffsetX" value="0.179" />
         <xacro:property name="wheelOffsetY" value="0.1815" />
@@ -51,20 +51,20 @@
         <link name="chassis">
             <collision>
-                <origin xyz="0 0 ${wheelRadius}" rpy="0 0 0"/>
+                <origin xyz="0 0 ${wheel_radius}" rpy="0 0 0"/>
                 <geometry>
-                  <box size="${chassisLength} ${chassisWidth} ${chassisHeight}"/>
+                  <box size="${chassis_length} ${chassis_width} ${chassis_height}"/>
                 </geometry>
             </collision>
             <visual>
-                <origin xyz="0 0 ${wheelRadius + chassisHeight/2}" rpy="0 0 0"/>
+                <origin xyz="0 0 ${wheel_radius + chassis_height/2}" rpy="0 0 0"/>
                 <geometry>
-                    <box size="${chassisLength} ${chassisWidth} ${chassisHeight}"/>
+                    <box size="${chassis_length} ${chassis_width} ${chassis_height}"/>
                 </geometry>
                 <material name="orange"/>
             </visual>
             <inertial>
-                <origin xyz="0 0 ${wheelRadius}" rpy="0 0 0"/>
-                <mass value="${chassisMass}"/>
-                <box_inertia m="${chassisMass}" x="${chassisLength}" y="${chassisWidth}" z="${chassisHeight}"/>
+                <origin xyz="0 0 ${wheel_radius}" rpy="0 0 0"/>
+                <mass value="${chassis_mass}"/>
+                <box_inertia m="${chassis_mass}" x="${chassis_length}" y="${chassis_width}" z="${chassis_height}"/>
             </inertial>
         </link>
@@ -76,6 +76,6 @@
                         lr_position="-1"
                         fr_position="1"
-                        wheel_radius="${wheelRadius}"
-                        wheel_mass="${wheelMass}"
+                        wheel_radius="${wheel_radius}"
+                        wheel_mass="${wheel_mass}"
                         axle_eff_limit="${front_axle_eff_limit}"
         />
@@ -84,6 +84,6 @@
                         lr_position="1"
                         fr_position="1"
-                        wheel_radius="${wheelRadius}"
-                        wheel_mass="${wheelMass}"
+                        wheel_radius="${wheel_radius}"
+                        wheel_mass="${wheel_mass}"
                         axle_eff_limit="${front_axle_eff_limit}"
         />
@@ -92,6 +92,6 @@
                     lr_position="1"
                     fr_position="-1"
-                    wheel_radius="${wheelRadius}"
-                    wheel_mass="${wheelMass}"
+                    wheel_radius="${wheel_radius}"
+                    wheel_mass="${wheel_mass}"
                     axle_eff_limit="${front_axle_eff_limit}"
         />
@@ -100,6 +100,6 @@
                     lr_position="-1"
                     fr_position="-1"
-                    wheel_radius="${wheelRadius}"
-                    wheel_mass="${wheelMass}"
+                    wheel_radius="${wheel_radius}"
+                    wheel_mass="${wheel_mass}"
                     axle_eff_limit="${front_axle_eff_limit}"
         />
@@ -109,5 +109,5 @@
     <!--
         <joint name="camera_joint" type="fixed">
-            <origin xyz="${-cameraSize+chassisLength/2} 0 ${cameraSize+wheelRadius+cameraSize/2}" rpy="0 0 0"/>
+            <origin xyz="${-cameraSize+chassis_length/2} 0 ${cameraSize+wheel_radius+cameraSize/2}" rpy="0 0 0"/>
             <parent link="chassis"/>
             <child link="camera"/>
@@ -137,5 +137,5 @@
         <joint name="hokuyo_joint" type="fixed">
             <axis xyz="0 1 0" />
-            <origin xyz="${-cameraSize+chassisLength/2} 0 ${cameraSize+wheelRadius + chassisHeight/2}" rpy="0 0 0"/>
+            <origin xyz="${-cameraSize+chassis_length/2} 0 ${cameraSize+wheel_radius + chassis_height/2}" rpy="0 0 0"/>
             <parent link="chassis"/>
             <child link="hokuyo_link"/>
